Commit message: 4-lidar TF frames as plain links/joints (VLP-16 macro drags meshes/gazebo baggage; suspected behavior-container CPU spin trigger)

File: container_patches/sensor_kit.xacro (robot description, xacro)
@@ -30,8 +30,11 @@
     </xacro:VLP-16>
     <!-- ROii 4-LiDAR suite: front/rear G32 (directional) + side rotating
-         Pandars. These create the lidar_front / lidar_rear / lidar_side_left /
-         lidar_side_right TF frames the CARLA mapping publishes into; without
-         them the concatenation node cannot transform to base_link. -->
-    <xacro:VLP-16 parent="sensor_kit_base_link" name="lidar_front" topic="/lidar_front_points" hz="10" samples="220" gpu="$(arg gpu)">
+         Pandars. PLAIN links+joints (no VLP-16 macro): the macro drags in
+         meshes/gazebo plugins; all we need is the TF frame for each lidar so
+         the concatenation node can transform clouds to base_link. -->
+    <link name="lidar_front"/>
+    <joint name="lidar_front_joint" type="fixed">
+      <parent link="sensor_kit_base_link"/>
+      <child link="lidar_front"/>
       <origin
         xyz="${calibration['sensor_kit_base_link']['lidar_front_base_link']['x']}
@@ -42,6 +45,9 @@
              ${calibration['sensor_kit_base_link']['lidar_front_base_link']['yaw']}"
       />
-    </xacro:VLP-16>
-    <xacro:VLP-16 parent="sensor_kit_base_link" name="lidar_rear" topic="/lidar_rear_points" hz="10" samples="220" gpu="$(arg gpu)">
+    </joint>
+    <link name="lidar_rear"/>
+    <joint name="lidar_rear_joint" type="fixed">
+      <parent link="sensor_kit_base_link"/>
+      <child link="lidar_rear"/>
       <origin
         xyz="${calibration['sensor_kit_base_link']['lidar_rear_base_link']['x']}
@@ -52,6 +58,9 @@
              ${calibration['sensor_kit_base_link']['lidar_rear_base_link']['yaw']}"
       />
-    </xacro:VLP-16>
-    <xacro:VLP-16 parent="sensor_kit_base_link" name="lidar_side_left" topic="/lidar_side_left_points" hz="10" samples="220" gpu="$(arg gpu)">
+    </joint>
+    <link name="lidar_side_left"/>
+    <joint name="lidar_side_left_joint" type="fixed">
+      <parent link="sensor_kit_base_link"/>
+      <child link="lidar_side_left"/>
       <origin
         xyz="${calibration['sensor_kit_base_link']['lidar_side_left_base_link']['x']}
@@ -62,6 +71,9 @@
              ${calibration['sensor_kit_base_link']['lidar_side_left_base_link']['yaw']}"
       />
-    </xacro:VLP-16>
-    <xacro:VLP-16 parent="sensor_kit_base_link" name="lidar_side_right" topic="/lidar_side_right_points" hz="10" samples="220" gpu="$(arg gpu)">
+    </joint>
+    <link name="lidar_side_right"/>
+    <joint name="lidar_side_right_joint" type="fixed">
+      <parent link="sensor_kit_base_link"/>
+      <child link="lidar_side_right"/>
       <origin
         xyz="${calibration['sensor_kit_base_link']['lidar_side_right_base_link']['x']}
@@ -72,5 +84,5 @@
              ${calibration['sensor_kit_base_link']['lidar_side_right_base_link']['yaw']}"
       />
-    </xacro:VLP-16>
+    </joint>
     <!-- cameras (6 for 360-degree coverage) -->
     <xacro:monocular_camera_macro

Commit message: Revert sensor_kit.xacro to VLP-16 version (plain-link URDF broke launch robot_description conversion)

File: container_patches/sensor_kit.xacro (robot description, xacro)
@@ -30,11 +30,8 @@
     </xacro:VLP-16>
     <!-- ROii 4-LiDAR suite: front/rear G32 (directional) + side rotating
-         Pandars. PLAIN links+joints (no VLP-16 macro): the macro drags in
-         meshes/gazebo plugins; all we need is the TF frame for each lidar so
-         the concatenation node can transform clouds to base_link. -->
-    <link name="lidar_front"/>
-    <joint name="lidar_front_joint" type="fixed">
-      <parent link="sensor_kit_base_link"/>
-      <child link="lidar_front"/>
+         Pandars. These create the lidar_front / lidar_rear / lidar_side_left /
+         lidar_side_right TF frames the CARLA mapping publishes into; without
+         them the concatenation node cannot transform to base_link. -->
+    <xacro:VLP-16 parent="sensor_kit_base_link" name="lidar_front" topic="/lidar_front_points" hz="10" samples="220" gpu="$(arg gpu)">
       <origin
         xyz="${calibration['sensor_kit_base_link']['lidar_front_base_link']['x']}
@@ -45,9 +42,6 @@
              ${calibration['sensor_kit_base_link']['lidar_front_base_link']['yaw']}"
       />
-    </joint>
-    <link name="lidar_rear"/>
-    <joint name="lidar_rear_joint" type="fixed">
-      <parent link="sensor_kit_base_link"/>
-      <child link="lidar_rear"/>
+    </xacro:VLP-16>
+    <xacro:VLP-16 parent="sensor_kit_base_link" name="lidar_rear" topic="/lidar_rear_points" hz="10" samples="220" gpu="$(arg gpu)">
       <origin
         xyz="${calibration['sensor_kit_base_link']['lidar_rear_base_link']['x']}
@@ -58,9 +52,6 @@
              ${calibration['sensor_kit_base_link']['lidar_rear_base_link']['yaw']}"
       />
-    </joint>
-    <link name="lidar_side_left"/>
-    <joint name="lidar_side_left_joint" type="fixed">
-      <parent link="sensor_kit_base_link"/>
-      <child link="lidar_side_left"/>
+    </xacro:VLP-16>
+    <xacro:VLP-16 parent="sensor_kit_base_link" name="lidar_side_left" topic="/lidar_side_left_points" hz="10" samples="220" gpu="$(arg gpu)">
       <origin
         xyz="${calibration['sensor_kit_base_link']['lidar_side_left_base_link']['x']}
@@ -71,9 +62,6 @@
              ${calibration['sensor_kit_base_link']['lidar_side_left_base_link']['yaw']}"
       />
-    </joint>
-    <link name="lidar_side_right"/>
-    <joint name="lidar_side_right_joint" type="fixed">
-      <parent link="sensor_kit_base_link"/>
-      <child link="lidar_side_right"/>
+    </xacro:VLP-16>
+    <xacro:VLP-16 parent="sensor_kit_base_link" name="lidar_side_right" topic="/lidar_side_right_points" hz="10" samples="220" gpu="$(arg gpu)">
       <origin
         xyz="${calibration['sensor_kit_base_link']['lidar_side_right_base_link']['x']}
@@ -84,5 +72,5 @@
              ${calibration['sensor_kit_base_link']['lidar_side_right_base_link']['yaw']}"
       />
-    </joint>
+    </xacro:VLP-16>
     <!-- cameras (6 for 360-degree coverage) -->
     <xacro:monocular_camera_macro
